File: IoP_plant_base.kicad_pcb (KiCad board)
At the start: 2 copper layers, 51.6 x 53.1 mm, 59 parts, among them IC1 HX711, J1 Conn_01x02, J2 Jack-DC, J4 Conn_01x02, J5 Conn_01x03, J6 Conn_01x02, J7 Conn_01x05, Q1 BC857C, Q2 IRLML6244, U1 NodeMCUv2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

Commit message: fixed inconsistent parts values, preliminary BOM created (missing Mouser part numbers)
Parts:
- C13, C7: value 100µF/6.3V -> 100uF/6.3V
- C14, C3: value 10µF -> 10uF
- C15: value 0.1µF -> 0.1uF
- C16: value 0.1uF -> 100nF
- C6: value 0.1µF -> 100nF
- C8, CFF1: value 1µF -> 1uF
Changed lines of the file:
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@@
-(kicad_pcb (version 20171130) (host pcbnew "(5.0.1)-rc2")
+(kicad_pcb (version 20171130) (host pcbnew "(6.0.0-rc1-dev-985-g576a0af29)")
   (general
     (thickness 1.6)
@@
     (zone_45_only yes)
     (trace_min 0.2)
-    (segment_width 0.2)
-    (edge_width 0.15)
     (via_size 0.8)
     (via_drill 0.4)
@@
     (uvia_min_size 0.2)
     (uvia_min_drill 0.1)
+    (edge_width 0.15)
+    (segment_width 0.2)
     (pcb_text_width 0.3)
     (pcb_text_size 1.5 1.5)
@@
       (effects (font (size 1 1) (thickness 0.15)))
     )
-    (fp_text value 0.1uF (at 0 1.43 180) (layer F.Fab)
+    (fp_text value 100nF (at 0 1.43 180) (layer F.Fab)
       (effects (font (size 1 1) (thickness 0.15)))
     )
@@
       (effects (font (size 1 1) (thickness 0.15)))
     )
-    (fp_text value 10µF (at 0 1.65) (layer F.Fab)
+    (fp_text value 10uF (at 0 1.65) (layer F.Fab)
       (effects (font (size 1 1) (thickness 0.15)))
     )
@@
       (effects (font (size 1 1) (thickness 0.15)))
     )
-    (fp_text value 10µF (at 0 1.65) (layer F.Fab)
+    (fp_text value 10uF (at 0 1.65) (layer F.Fab)
       (effects (font (size 1 1) (thickness 0.15)))
     )
@@
       (effects (font (size 1 1) (thickness 0.15)))
     )
-    (fp_text value 0.1µF (at 0 1.43 90) (layer F.Fab)
+    (fp_text value 0.1uF (at 0 1.43 90) (layer F.Fab)
       (effects (font (size 1 1) (thickness 0.15)))
     )
@@
       (effects (font (size 1 1) (thickness 0.15)))
     )
-    (fp_text value 0.1µF (at 0 1.43 180) (layer F.Fab)
+    (fp_text value 100nF (at 0 1.43 180) (layer F.Fab)
       (effects (font (size 1 1) (thickness 0.15)))
     )
@@
       (effects (font (size 1 1) (thickness 0.15)))
     )
-    (fp_text value 1µF (at 0 1.43 270) (layer F.Fab)
+    (fp_text value 1uF (at 0 1.43 270) (layer F.Fab)
       (effects (font (size 1 1) (thickness 0.15)))
     )
@@
       (effects (font (size 1 1) (thickness 0.15)))
     )
-    (fp_text value 100µF/6.3V (at 0 2.35 180) (layer F.Fab)
+    (fp_text value 100uF/6.3V (at 0 2.35 180) (layer F.Fab)
       (effects (font (size 1 1) (thickness 0.15)))
     )
@@
       (effects (font (size 1 1) (thickness 0.15)))
     )
-    (fp_text value 100µF/6.3V (at 0 2.35) (layer F.Fab)
+    (fp_text value 100uF/6.3V (at 0 2.35) (layer F.Fab)
       (effects (font (size 1 1) (thickness 0.15)))
     )
@@
       (effects (font (size 1 1) (thickness 0.15)))
     )
-    (fp_text value 1µF (at 0 1.43 270) (layer F.Fab)
+    (fp_text value 1uF (at 0 1.43 270) (layer F.Fab)
       (effects (font (size 1 1) (thickness 0.15)))
     )
@@
     )
   )
-  (module kicad_art:nyantronics_logo (layer F.Cu)
+  (module kicad_art:nyantronics_logo locked (layer F.Cu)
     (at 117.38102 105.25506 90)
     (fp_text reference G*** (at 0 0 90) (layer F.SilkS) hide
@@
       (xy -0.939992 -1.772491) (xy -0.500661 -1.775565) (xy -0.047814 -1.77677) (xy 0.406741 -1.776106)) (layer F.SilkS) (width 0.01))
   )
-  (module kicad_art:kitten_paw_prints (layer F.Cu)
+  (module kicad_art:kitten_paw_prints locked (layer F.Cu)
     (at 109.36224 106.55808 90)
     (fp_text reference G*** (at 0 0 90) (layer F.SilkS) hide
@@
   (segment (start 122.682 121.4628) (end 122.2248 121.92) (width 0.3) (layer F.Cu) (net 34))
   (segment (start 122.682 115.6208) (end 122.682 121.4628) (width 0.3) (layer F.Cu) (net 34))
-  (segment (start 116.332 93.901) (end 116.332 109.2708) (width 0.3) (layer F.Cu) (net 34))
+  (segment (start 116.332 93.901) (end 116.332 109.2708) (width 0.3) (layer F.Cu) (net 34) (status 40000))
   (segment (start 116.332 109.2708) (end 122.682 115.6208) (width 0.3) (layer F.Cu) (net 34))
   (segment (start 124.4542 85.1406) (end 124.4612 85.1336) (width 0.3) (layer F.Cu) (net 35) (status 30))

Commit message: updated BOM info according to Mouser order. Note: consider migrating to ME2149F SO8 for next rev. (higher current, ~30ct vs. 1.15€)
Parts:
- C1, C16, C17, C18, C19, C6: value 100nF -> 100nF/50V
- C10, C11: value 10nF -> 10nF/50V
- C12, C14, C3: value 10uF -> 10uF/16V
- C15, C9: value 0.1uF -> 100nF/50V
- C5: value 4.7uF -> 4.7uF/25V
- C8, CFF1: value 1uF -> 1uF/50V
- R10, R11, R14, R4, R5: value 100 -> 100R
Changed lines of the file:
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@@
       (effects (font (size 1 1) (thickness 0.15)))
     )
-    (fp_text value 100 (at 0 1.43) (layer F.Fab)
+    (fp_text value 100R (at 0 1.43) (layer F.Fab)
       (effects (font (size 1 1) (thickness 0.15)))
     )
@@
       (effects (font (size 1 1) (thickness 0.15)))
     )
-    (fp_text value 100nF (at 0 1.43 180) (layer F.Fab)
+    (fp_text value 100nF/50V (at 0 1.43 180) (layer F.Fab)
       (effects (font (size 1 1) (thickness 0.15)))
     )
@@
       (effects (font (size 1 1) (thickness 0.15)))
     )
-    (fp_text value 100nF (at 0 1.43 90) (layer F.Fab)
+    (fp_text value 100nF/50V (at 0 1.43 90) (layer F.Fab)
       (effects (font (size 1 1) (thickness 0.15)))
     )
@@
       (effects (font (size 1 1) (thickness 0.15)))
     )
-    (fp_text value 100nF (at 0 1.43 270) (layer F.Fab)
+    (fp_text value 100nF/50V (at 0 1.43 270) (layer F.Fab)
       (effects (font (size 1 1) (thickness 0.15)))
     )
@@
       (effects (font (size 1 1) (thickness 0.15)))
     )
-    (fp_text value 4.7uF (at 0 1.65) (layer F.Fab)
+    (fp_text value 4.7uF/25V (at 0 1.65) (layer F.Fab)
       (effects (font (size 1 1) (thickness 0.15)))
     )
@@
       (effects (font (size 1 1) (thickness 0.15)))
     )
-    (fp_text value 100nF (at 0 1.43 180) (layer F.Fab)
+    (fp_text value 100nF/50V (at 0 1.43 180) (layer F.Fab)
       (effects (font (size 1 1) (thickness 0.15)))
     )
@@
       (effects (font (size 1 1) (thickness 0.15)))
     )
-    (fp_text value 100nF (at 0 1.43 180) (layer F.Fab)
+    (fp_text value 100nF/50V (at 0 1.43 180) (layer F.Fab)
       (effects (font (size 1 1) (thickness 0.15)))
     )
@@
       (effects (font (size 1 1) (thickness 0.15)))
     )
-    (fp_text value 10uF (at 0 1.65) (layer F.Fab)
+    (fp_text value 10uF/16V (at 0 1.65) (layer F.Fab)
       (effects (font (size 1 1) (thickness 0.15)))
     )
@@
       (effects (font (size 1 1) (thickness 0.15)))
     )
-    (fp_text value 10uF (at 0 1.65 180) (layer F.Fab)
+    (fp_text value 10uF/16V (at 0 1.65 180) (layer F.Fab)
       (effects (font (size 1 1) (thickness 0.15)))
     )
@@
       (effects (font (size 1 1) (thickness 0.15)))
     )
-    (fp_text value 10uF (at 0 1.65) (layer F.Fab)
+    (fp_text value 10uF/16V (at 0 1.65) (layer F.Fab)
       (effects (font (size 1 1) (thickness 0.15)))
     )
@@
       (effects (font (size 1 1) (thickness 0.15)))
     )
-    (fp_text value 0.1uF (at 0 1.43 90) (layer F.Fab)
+    (fp_text value 100nF/50V (at 0 1.43 90) (layer F.Fab)
       (effects (font (size 1 1) (thickness 0.15)))
     )
@@
       (effects (font (size 1 1) (thickness 0.15)))
     )
-    (fp_text value 100nF (at 0 1.43 180) (layer F.Fab)
+    (fp_text value 100nF/50V (at 0 1.43 180) (layer F.Fab)
       (effects (font (size 1 1) (thickness 0.15)))
     )
@@
       (effects (font (size 1 1) (thickness 0.15)))
     )
-    (fp_text value 1uF (at 0 1.43 270) (layer F.Fab)
+    (fp_text value 1uF/50V (at 0 1.43 270) (layer F.Fab)
       (effects (font (size 1 1) (thickness 0.15)))
     )
@@
       (effects (font (size 1 1) (thickness 0.15)))
     )
-    (fp_text value 0.1uF (at 0 1.43 180) (layer F.Fab)
+    (fp_text value 100nF/50V (at 0 1.43 180) (layer F.Fab)
       (effects (font (size 1 1) (thickness 0.15)))
     )
@@
       (effects (font (size 1 1) (thickness 0.15)))
     )
-    (fp_text value 100 (at 3.3275 0) (layer F.Fab)
+    (fp_text value 100R (at 3.3275 0) (layer F.Fab)
       (effects (font (size 1 1) (thickness 0.15)))
     )
@@
       (effects (font (size 1 1) (thickness 0.15)))
     )
-    (fp_text value 100 (at -3.0735 -0.127) (layer F.Fab)
+    (fp_text value 100R (at -3.0735 -0.127) (layer F.Fab)
       (effects (font (size 1 1) (thickness 0.15)))
     )
@@
       (effects (font (size 1 1) (thickness 0.15)))
     )
-    (fp_text value 100 (at 0 1.43 270) (layer F.Fab)
+    (fp_text value 100R (at 0 1.43 270) (layer F.Fab)
       (effects (font (size 1 1) (thickness 0.15)))
     )
@@
       (effects (font (size 1 1) (thickness 0.15)))
     )
-    (fp_text value 100 (at 0 1.43 270) (layer F.Fab)
+    (fp_text value 100R (at 0 1.43 270) (layer F.Fab)
       (effects (font (size 1 1) (thickness 0.15)))
     )
@@
       (effects (font (size 1 1) (thickness 0.15)))
     )
-    (fp_text value 1uF (at 0 1.43 270) (layer F.Fab)
+    (fp_text value 1uF/50V (at 0 1.43 270) (layer F.Fab)
       (effects (font (size 1 1) (thickness 0.15)))
     )
@@
       (effects (font (size 1 1) (thickness 0.15)))
     )
-    (fp_text value 10nF (at 3.5305 0) (layer F.Fab)
+    (fp_text value 10nF/50V (at 3.5305 0) (layer F.Fab)
       (effects (font (size 1 1) (thickness 0.15)))
     )
@@
       (effects (font (size 1 1) (thickness 0.15)))
     )
-    (fp_text value 10nF (at 3.4545 0.127 180) (layer F.Fab)
-      (effects (font (size 1 1) (thickness 0.15)))
-    )
+    (fp_text value 10nF/50V (at 3.4545 0.127 180) (layer F.Fab)
+      (effects (font (size 1 1) (thickness 0.15)))
+    )
